File: Temp-Humidity-Monitor-FINAL.kicad_pcb (KiCad board)
At the start: 2 copper layers, 106 x 51.5 mm, 17 parts, among them U1 ARDUINO_NANO, U2 DHT22, U3 ER_OLEDM0.91_1x-I2C

Commit message: Add files via upload
Fixed PCB with no Clearance Problem
Routing:
- net Net-(U1-+5V): track 58.2 -> 60.3 mm
